File: hardware/current-monitor.sch (KiCad schematic (older format))
At the start: 57 parts, among them J1 SENSE, J2 BATTERY, J3 LCD5110, J4 UART, J5 SWD, J6 JTAG, Q1 MUN5314DW1, U1 AP2210K-3.3, U2 MKL03Z8VFK4, U3 MCP6V71U, U4 MCP6001U

Commit message: start redesign
Parts:
- removed J3: LCD5110, libs:CONN-2x4-1.0-PTH-SHROUD, symbol LCD5110
- removed J4: UART, libs:CONN-4-2.54-0.8-PTH, symbol CONN-4
- removed Q1: MUN5314DW1, libs:SOT-23-6, symbol MUN53
- removed R11, R4: 6.81k, libs:SMD-1608, symbol R
- removed R12, R5: 536, libs:SMD-1608, symbol R
- removed U2: MKL03Z8VFK4, libs:qfn-24-4x4, symbol MKL03ZxxVFK4
- added C? (x2): 0.1u, libs:SMD-1608, symbol C
- added C? (x10): 1u, symbol C
- added C?: 10u, symbol C
- added C? (x2): 2.2u, libs:SMD-2012, symbol C
- added D?: BAV70, symbol D-DUAL-COMMON-CATHODE-SOT-23
- added F?: 0ZCJ0110FF2E, symbol FUSE
- added J?: ERC12864-1, symbol ERC12864-1
- added J?: LCD_BL, symbol CONN-2
- added J?: USB-MICROB, symbol USB-MICROB
- added J?: DB9, symbol DB9
- added L? (x2): 22u, symbol L
- added Q?: 2N2222, symbol NPN
- added R? (x2): 33, libs:SMD-1608, symbol Rs
- added R?: 1k, libs:SMD-1608, symbol R
- added R? (x4): 100k, libs:SMD-1608, symbol R
- added R? (x2): 499, libs:SMD-1608, symbol R
- added R? (x2): 1k, libs:SMD-1608, symbol Rs
- added U?: MKL27ZxxVFM4, symbol MKL27ZxxVFM4
- J1: BOM 1-2834021-2 -> (none)
- R17: value 1M -> 10k; BOM MCT06030C1004FP500 -> (none)
- R18: value 10k -> 1k; BOM RR0816P-103-D -> (none)
- R19, R20: value 499 -> 1k; BOM RR0816P-4990-D-68A -> (none)
- R3, R7: value 1M -> 100k; BOM MCT06030C1004FP500 -> (none)
- U3: value MCP6V71U -> MCP6V81U; footprint libs:SOT-23-5 -> libs:SC-70; BOM MCP6V71UT-E/LTY -> MCP6V81UT-E/LTY
Connections:
- net labels added: BAT_SENSE, DB9_USR1, DB9_USR2, LCD_CLK, LCD_MOSI, USB_DM, USB_DP, VUSB, ~LCD_RES
- net labels removed: MISO, MOSI, SCLK, SD_DET, ~SD_CS
- wire segments 139 -> 249
- no-connect marks 11 -> 13
Other:
- note added: "11mV"
- note added: "494R impedance"
- note added: "9uV offset V RTI\n9mV offset V RTO"
- note added: "DB9 Serial"
- note added: "Display Backlight"
- note added: "USB"
- note removed: "497R impedance"
- note removed: "87mV"
- note removed: "8uV offset V RTI\n80mV offset V RTO"
- moved on the sheet: C1, C10, C2, C3, C5, C6, C9, J1, J2, J5, J6, R13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

Commit message: redesign for v1 r1
Parts:
- removed C?: 10u, symbol C
- removed J6: JTAG, libs:CONN-2x5-1.27-SMT, symbol JTAG
- removed J?: DB9, symbol DB9
- removed R?: 100k, libs:SMD-1608, symbol R
- removed S3: slide-SPDT, libs:SLIDE-1P2T-SIDE-PTH, symbol slide-SPDT
- added C25, C28: 2.2u 16V, libs:SMD-2012, symbol C
- added J6: AUX, libs:CONN-2x4-1.0-PTH-RIGHT-SHROUD, symbol CONN-2x4
- added Q2: 2N2222, libs:SOT-23-BJT, symbol NPN
- added S1: POWER, libs:SWITCH-8x8-DPDT, symbol button-DPDT
- added U5, U6: NUP4114, libs:SOT-23-6, symbol NUP4114
- C16, C17, C18, C19, C20, C21, C22, C23, C24, C26: renamed from C?; footprint (none) -> libs:SMD-1608
- D1: renamed from D?; footprint (none) -> libs:SOT-23
- F1: renamed from F?; value 0ZCJ0110FF2E -> 1.1A; footprint (none) -> libs:SMD-3216; BOM (none) -> 0ZCJ0110FF2E
- J1: footprint libs:TERM-2-2.5 -> libs:JST-XH-2-PTH-TOP
- J3: renamed from J?; footprint (none) -> libs:ER-CON30HB-1
- J4: renamed from J?; footprint (none) -> libs:USB-MICRO-B-FCI-10103594
- J5: renamed from J?; footprint (none) -> libs:ER-CON2.0-2P-SMD
- J7: renamed from J5; footprint libs:CONN-4-2.54-0.8-PTH -> libs:CONN-5-2.54-1.0-PTH; symbol CONN-4 -> CONN-5
- L1, L2: renamed from L?; footprint (none) -> libs:SMD-1608
- Q1: renamed from Q?; footprint (none) -> libs:SOT-23-BJT
- R13: renamed from R21; symbol Rs -> R
- R2: renamed from R17; value 10k -> 100k
- R22: symbol Rs -> R
- R25: renamed from R13; value 1k -> 120; symbol R -> Rs
- R3: renamed from R18; value 1k -> 10k
- U2: renamed from U3; footprint libs:SC-70 -> libs:SOT-23-5; BOM MCP6V81UT-E/LTY -> MCP6V81UT-E/OT
- U4: renamed from U?; footprint (none) -> libs:MKL27ZxxVFM4
- gave numbers to parts that had none: 14
- renumbered C10 to C1, C5 to C12, C6 to C15, C1 to C2, C9 to C27, C2 to C3, C3 to C4, C4 to C5, C8 to C6, C11 to C7, C7 to C8, C12 to C9, R6 to R10, R7 to R11, R8 to R12, R9 to R17, R10 to R18, R14 to R19, R15 to R20, R16 to R21, R19 to R27, R20 to R29, R25 to R4, R2 to R8, R3 to R9, S1 to S2, S2 to S3, TP7 to TP1, TP8 to TP2, TP4 to TP3, TP1 to TP4, TP2 to TP5, TP5 to TP6, TP6 to TP7, TP3 to TP8, U4 to U3
Connections:
- net labels added: AUX_USR1, AUX_USR2, LCD_LED, VIN
- net labels removed: DB9_USR1, DB9_USR2, ~LCD_LED
- wire segments 249 -> 204
- no-connect marks 13 -> 16
Other:
- note added: "497R impedance"
- note added: "6mV"
- note added: "Debug Connector"
- note added: "I_LED =~~ 0.67/R25"
- note added: "Serial and Aux"
- note removed: "DB9 Serial"
- note removed: "Debug Connectors"
- moved on the sheet: C1, C2, C27, C3, C4, D1, J2, J4, J5, L1, L2, Q1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

Commit message: BOM for schematic
Parts:
- C10, C13, C3: value 2.2u -> 2.2u 16V
- C16, C17, C18, C19, C20, C21, C22, C23, C24, C26: BOM (none) -> CL10A105KO8NNNC
- D1: value BAV70 -> BAT54; BOM (none) -> BAT54CLT1G
- J1: BOM (none) -> B2B-XH-A(LF)(SN)
- J4: BOM (none) -> 10103594-0001LF
- J6: BOM (none) -> 75867-132LF
- Q1, Q2: BOM (none) -> MMBT2222ALT3G
- R11, R14, R2, R5, R6, R9: BOM (none) -> RR0816P-104-D
- R25: BOM RR0816P-102-D -> (none)
- R3: BOM (none) -> RR0816P-103-D
- S1: BOM (none) -> TL2201EEYA
Changed lines of the file:
@@
 F 2 "libs:SMD-1608" H 2185 3440 60  0001 C CNN
 F 3 "" H 2185 3440 60  0000 C CNN
+F 4 "RR0816P-104-D" H 2050 3600 60  0001 C CNN "BOM"
 	1    2050 3600
 	0    1    1    0
@@
 F 2 "libs:SMD-1608" H 10385 5740 60  0001 C CNN
 F 3 "" H 10385 5740 60  0000 C CNN
-F 4 "RR0816P-102-D" H 10250 5900 60  0001 C CNN "BOM"
 	1    10250 5900
 	1    0    0    -1
@@
 F 2 "libs:SMD-1608" H 2185 2140 60  0001 C CNN
 F 3 "" H 2185 2140 60  0000 C CNN
+F 4 "RR0816P-104-D" H 2050 2300 60  0001 C CNN "BOM"
 	1    2050 2300
 	0    1    1    0
@@
 P 9050 1100
 F 0 "C3" H 9123 1046 50  0000 L CNN
-F 1 "2.2u" H 9123 955 50  0000 L CNN
+F 1 "2.2u 16V" H 9123 955 50  0000 L CNN
 F 2 "libs:SMD-2012" H 8950 1250 60  0001 C CNN
 F 3 "" H 8950 1250 60  0000 C CNN
@@
 F 2 "libs:SMD-1608" H 6235 1190 60  0001 C CNN
 F 3 "" H 6235 1190 60  0000 C CNN
+F 4 "RR0816P-103-D" H 6100 1350 60  0001 C CNN "BOM"
 	1    6100 1350
 	-1   0    0    -1
@@
 F 2 "libs:SMD-1608" H 9650 2800 60  0001 C CNN
 F 3 "" H 9650 2800 60  0000 C CNN
+F 4 "CL10A105KO8NNNC" H 9750 2650 60  0001 C CNN "BOM"
 	1    9750 2650
 	1    0    0    -1
@@
 F 2 "libs:SMD-1608" H 9650 3000 60  0001 C CNN
 F 3 "" H 9650 3000 60  0000 C CNN
+F 4 "CL10A105KO8NNNC" H 9750 2850 60  0001 C CNN "BOM"
 	1    9750 2850
 	1    0    0    -1
@@
 F 2 "libs:SMD-1608" H 9650 3300 60  0001 C CNN
 F 3 "" H 9650 3300 60  0000 C CNN
+F 4 "CL10A105KO8NNNC" H 9750 3150 60  0001 C CNN "BOM"
 	1    9750 3150
 	1    0    0    -1
@@
 F 2 "libs:SMD-1608" H 10450 3700 60  0001 C CNN
 F 3 "" H 10450 3700 60  0000 C CNN
+F 4 "CL10A105KO8NNNC" H 10550 3550 60  0001 C CNN "BOM"
 	1    10550 3550
 	0    -1   1    0
@@
 F 2 "libs:SMD-1608" H 10250 3800 60  0001 C CNN
 F 3 "" H 10250 3800 60  0000 C CNN
+F 4 "CL10A105KO8NNNC" H 10350 3650 60  0001 C CNN "BOM"
 	1    10350 3650
 	0    -1   1    0
@@
 F 2 "libs:SMD-1608" H 10050 3900 60  0001 C CNN
 F 3 "" H 10050 3900 60  0000 C CNN
+F 4 "CL10A105KO8NNNC" H 10150 3750 60  0001 C CNN "BOM"
 	1    10150 3750
 	0    -1   1    0
@@
 F 2 "libs:SMD-1608" H 9850 4000 60  0001 C CNN
 F 3 "" H 9850 4000 60  0000 C CNN
+F 4 "CL10A105KO8NNNC" H 9950 3850 60  0001 C CNN "BOM"
 	1    9950 3850
 	0    -1   1    0
@@
 F 2 "libs:SMD-1608" H 9650 4100 60  0001 C CNN
 F 3 "" H 9650 4100 60  0000 C CNN
+F 4 "CL10A105KO8NNNC" H 9750 3950 60  0001 C CNN "BOM"
 	1    9750 3950
 	0    -1   1    0
@@
 F 2 "libs:SMD-1608" H 9950 2700 60  0001 C CNN
 F 3 "" H 9950 2700 60  0000 C CNN
+F 4 "CL10A105KO8NNNC" H 10050 2550 60  0001 C CNN "BOM"
 	1    10050 2550
 	1    0    0    -1
@@
 F 2 "libs:SMD-1608" H 8350 4200 60  0001 C CNN
 F 3 "" H 8350 4200 60  0000 C CNN
+F 4 "CL10A105KO8NNNC" H 8450 4050 60  0001 C CNN "BOM"
 	1    8450 4050
 	1    0    0    -1
@@
 P 4600 3500
 F 0 "C10" H 4673 3446 50  0000 L CNN
-F 1 "2.2u" H 4673 3355 50  0000 L CNN
+F 1 "2.2u 16V" H 4673 3355 50  0000 L CNN
 F 2 "libs:SMD-2012" H 4500 3650 60  0001 C CNN
 F 3 "" H 4500 3650 60  0000 C CNN
@@
 P 4700 4100
 F 0 "C13" H 4773 4046 50  0000 L CNN
-F 1 "2.2u" H 4773 3955 50  0000 L CNN
+F 1 "2.2u 16V" H 4773 3955 50  0000 L CNN
 F 2 "libs:SMD-2012" H 4600 4250 60  0001 C CNN
 F 3 "" H 4600 4250 60  0000 C CNN
@@
 F 2 "libs:SMD-1608" H 6235 990 60  0001 C CNN
 F 3 "" H 6235 990 60  0000 C CNN
+F 4 "RR0816P-104-D" H 6100 1150 60  0001 C CNN "BOM"
 	1    6100 1150
 	-1   0    0    -1
@@
 F 2 "libs:SOT-23-BJT" H 10250 5750 60  0001 C CNN
 F 3 "" H 10250 5750 60  0000 C CNN
+F 4 "MMBT2222ALT3G" H 10250 5750 60  0001 C CNN "BOM"
 	1    10250 5750
 	1    0    0    -1
@@
 P 7000 1050
 F 0 "D1" V 6785 925 50  0000 C CNN
-F 1 "BAV70" V 6694 925 50  0000 C CNN
+F 1 "BAT54" V 6694 925 50  0000 C CNN
 F 2 "libs:SOT-23" H 7000 900 60  0001 C CNN
 F 3 "" H 7000 900 60  0000 C CNN
+F 4 "BAT54CLT1G" H 7000 1050 60  0001 C CNN "BOM"
 	1    7000 1050
 	0    -1   -1   0
@@
 F 2 "libs:USB-MICRO-B-FCI-10103594" H 4900 5250 60  0001 C CNN
 F 3 "" H 4900 5250 60  0000 C CNN
+F 4 "10103594-0001LF" H 4800 5600 60  0001 C CNN "BOM"
 	1    4800 5600
 	1    0    0    -1
@@
 F 2 "libs:SMD-1608" H 3368 1709 60  0001 L CNN
 F 3 "" H 3435 1790 60  0000 C CNN
+F 4 "RR0816P-104-D" H 3300 1950 60  0001 C CNN "BOM"
 	1    3300 1950
 	1    0    0    -1
@@
 F 2 "libs:SMD-1608" H 3468 1709 60  0001 L CNN
 F 3 "" H 3535 1790 60  0000 C CNN
+F 4 "RR0816P-104-D" H 3400 1950 60  0001 C CNN "BOM"
 	1    3400 1950
 	1    0    0    -1
@@
 F 2 "libs:SMD-1608" H 3368 4009 60  0001 L CNN
 F 3 "" H 3435 4090 60  0000 C CNN
+F 4 "RR0816P-104-D" H 3300 4250 60  0001 C CNN "BOM"
 	1    3300 4250
 	-1   0    0    -1
@@
 F 2 "libs:SWITCH-8x8-DPDT" H 5200 1350 60  0001 C CNN
 F 3 "" H 5200 1350 60  0001 C CNN
+F 4 "TL2201EEYA" H 5200 1350 60  0001 C CNN "BOM"
 	1    5200 1350
 	0    1    1    0
@@
 F 2 "libs:CONN-2x4-1.0-PTH-RIGHT-SHROUD" H 2750 7850 50  0001 C CNN
 F 3 "" H 2750 7850 50  0000 C CNN
+F 4 "75867-132LF" H 2150 7050 60  0001 C CNN "BOM"
 	1    2150 7050
 	1    0    0    -1
@@
 F 2 "libs:JST-XH-2-PTH-TOP" H 1850 1050 60  0001 C CNN
 F 3 "" H 1850 1050 60  0000 C CNN
+F 4 "B2B-XH-A(LF)(SN)" H 1750 1250 60  0001 C CNN "BOM"
 	1    1750 1250
 	-1   0    0    -1
@@
 F 2 "libs:SOT-23-BJT" H 9850 5900 60  0001 C CNN
 F 3 "" H 9850 5900 60  0000 C CNN
+F 4 "MMBT2222ALT3G" H 9850 5900 60  0001 C CNN "BOM"
 	1    9850 5900
 	-1   0    0    -1
